File: v1 files/petr/petr.kicad_pcb (KiCad board)
At the start: 2 copper layers, 38.5 x 55.1 mm, 5 parts

Commit message: update
Parts:
- removed the REF** at (158.5, 91.8) (x2)
- added G***: LOGO, img:v5cucuBacking, F.Cu at (159.9, 85.0)
- added G***: LOGO, img:v5cucuFront, F.Cu at (159.9, 85.0)
Routing:
- net (no net): track 856.0 -> 0.00 mm, vias 17 -> 0
- removed copper zone on F.Cu, net (none)
Other:
- board text added: "#001"
- board text removed: "#002"
